File: adrover_pcb.kicad_pcb (KiCad board)
At the start: 2 copper layers, 11 parts, among them J1 BATTERY, J2 CONTROLLER, J3 RIGHT_M, J4 LEFT_M, J5 RIGHT_D, J6 LEFT_D, J7 RIGHT_D_POWER, J8 LEFT_D_POWER, U1 LM7805_TO220

Commit message: -
Parts:
- moved C1 52.7 mm to (148.6, 124.7)
- moved U1 43.8 mm to (150.9, 94.8), turned to 90 degrees
- moved J3 37.7 mm to (211.7, 97.3), turned to 180 degrees
- moved J4 35.2 mm to (85.3, 97.4), turned to 180 degrees
- moved C2 28.4 mm to (162.2, 89.6), turned to -90 degrees
- moved J6 20.9 mm to (115.0, 68.8), turned to 180 degrees
- moved J7 13.7 mm to (193.3, 117.1), turned to -90 degrees
- moved J8 6.58 mm to (99.2, 114.9), turned to -90 degrees
- moved J1 6.41 mm to (145.4, 136.9)
- moved J5 2.58 mm to (206.2, 57.5)
Routing:
- net /GND: track 0.00 -> 252.1 mm
- net /5V: track 0.00 -> 126.6 mm
- net /12V: track 0.00 -> 51.1 mm
